Commit message: updated meshes

File: scara_description/urdf/scara_dxl.urdf (robot description, URDF)
Before this commit: robot scara, 6 links, 5 joints
Links:
- added link pen; collision mesh filename=package://scara_description/meshes/scaradxl_pen.dae scale=0.001 0.001 0.001; visual mesh filename=package://scara_description/meshes/scaradxl_pen.dae scale=0.001 0.001 0.001
- link base_link: geometry collision mesh filename=package://scara_description/meshes/scaradxl_base.dae scale=0.001 0.001 0.001; visual mesh filename=package://scara_description/meshes/scaradxl_base.dae scale=0.001 0.001 0.001
- link link1: geometry collision mesh filename=package://scara_description/meshes/scaradxl_link1.dae scale=0.001 0.001 0.001; visual mesh filename=package://scara_description/meshes/scaradxl_link1.dae scale=0.001 0.001 0.001
- link link2: geometry collision mesh filename=package://scara_description/meshes/scaradxl_link2.dae scale=0.001 0.001 0.001; visual mesh filename=package://scara_description/meshes/scaradxl_link2.dae scale=0.001 0.001 0.001
- link link3: geometry collision mesh filename=package://scara_description/meshes/scaradxl_link3.dae scale=0.001 0.001 0.001; visual mesh filename=package://scara_description/meshes/scaradxl_link3.dae scale=0.001 0.001 0.001
Joints:
- removed joint tool02link3
- added joint pen2link3: type fixed, parent link3, child pen, origin xyz=0.1 0 0 rpy=0 0 0, axis 0 0 0
- added joint tool02pen: type fixed, parent pen, child tool0, origin xyz=0 0 0.1 rpy=0 0 0, axis 0 0 0
- joint joint1: origin xyz=0.0 0.0 0.020 rpy=0 0 0 -> xyz=0.0 0.0 0.14 rpy=0 0 0
- joint joint2: origin xyz=0.0 0.0743 0.0 rpy=0 0 0.0 -> xyz=0.0743 0.0 0.0 rpy=0 0 0.0
- joint joint3: origin xyz=0.0 0.1 0.0 rpy=0 0 0.0 -> xyz=0.1 0.0 0.0 rpy=0 0 0.0
