Commit message: Enhances gazebo part.

File: scara_description/config/scara.gazebo.config.xacro (robot description, xacro)
@@ -7,6 +7,6 @@
     <xacro:include filename="$(find scara_description)/config/materials.urdf" />
     <!-- Import scara ros2_control description -->
-    <xacro:include filename="$(find scara_description)/ros2_control/scara.ros2_control.urdf" />
+    <xacro:include filename="$(find scara_description)/ros2_control/scara.gazebo.ros2_control.urdf" />
     <!-- Import all Gazebo-customization elements -->
-    <!-- <xacro:include filename="$(find scara_description)/gazebo/scara.gazebo.xacro" /> -->
+    <xacro:include filename="$(find scara_description)/gazebo/scara.gazebo.xacro" />
 </robot>

File: scara_description/gazebo/scara.gazebo.xacro (robot description, xacro)
@@ -1,36 +1,36 @@
 <?xml version="1.0"?>
 <robot xmlns:xacro="http://www.ros.org/wiki/xacro" name="scara">
-    <!-- ros_control plugin -->
-    <gazebo>
-      <plugin filename="libgazebo_ros2_control.so" name="gazebo_ros2_control">
-        <parameters>$(find scara_description)/config/scara_controllers.yaml</parameters>
-        <robot_param_node>robot_state_publisher</robot_param_node>
-      </plugin>
-    </gazebo>
-    <!-- Used for fixing robot -->
-    <gazebo reference="world">
-        <static>true</static>
-    </gazebo>
-    <!-- color -->
-    <gazebo reference="base_link">
-      <material>Gazebo/Blue</material>
-    </gazebo>
-    <gazebo reference="revolute1">
-      <material>Gazebo/Green</material>
-    </gazebo>
-    <gazebo reference="link1">
-      <material>Gazebo/Blue</material>
-    </gazebo>
-    <gazebo reference="revolute2">
-      <material>Gazebo/Green</material>
-    </gazebo>
-    <gazebo reference="link2">
-      <material>Gazebo/Blue</material>
-    </gazebo>
-    <gazebo reference="prismatic3">
-      <material>Gazebo/Orange</material>
-    </gazebo>
-    <gazebo reference="link3">
-      <material>Gazebo/Blue</material>
-    </gazebo>
+  <!-- ros_control plugin -->
+  <gazebo>
+    <plugin filename="libgazebo_ros2_control.so" name="gazebo_ros2_control">
+      <parameters>$(find scara_description)/config/scara_controllers.yaml</parameters>
+      <robot_param_node>robot_state_publisher</robot_param_node>
+    </plugin>
+  </gazebo>
+  <!-- Used for fixing robot -->
+  <gazebo reference="world">
+    <static>true</static>
+  </gazebo>
+  <!-- color -->
+  <gazebo reference="base_link">
+    <material>Gazebo/Blue</material>
+  </gazebo>
+  <gazebo reference="revolute1">
+    <material>Gazebo/Green</material>
+  </gazebo>
+  <gazebo reference="link1">
+    <material>Gazebo/Blue</material>
+  </gazebo>
+  <gazebo reference="revolute2">
+    <material>Gazebo/Green</material>
+  </gazebo>
+  <gazebo reference="link2">
+    <material>Gazebo/Blue</material>
+  </gazebo>
+  <gazebo reference="prismatic3">
+    <material>Gazebo/Orange</material>
+  </gazebo>
+  <gazebo reference="link3">
+    <material>Gazebo/Blue</material>
+  </gazebo>
 </robot>
